Commit message: update robot model

File: src/my_robot_description/urdf/my_robot.urdf (robot description, URDF)
Before this commit: robot my_robot, 4 links, 3 joints
Joints:
- joint left_wheel_joint: limit lower=-inf upper=inf -> lower=-3.14 upper=3.14 effort=100.0 velocity=1.0; origin xyz=0.1 0 -0.05 rpy=0 0 0 -> xyz=0.1 0 0.05 rpy=0 0 0
- joint right_wheel_joint: limit lower=-inf upper=inf -> lower=-3.14 upper=3.14 effort=100.0 velocity=1.0; origin xyz=0.1 0 0.05 rpy=0 0 0 -> xyz=0.1 0 -0.05 rpy=0 0 0
